Commit message: gazebo marche sur z en global
le node fonctionne mais le wrench est appliqué uniquement sur le repère monde-> il faut convertir notre thrust en force dans le repère monde

File: controleDrone/urdf/drone.urdf (robot description, URDF)
Before this commit: robot myDrone, 5 links, 4 joints
Links:
- link BL: geometry visual cylinder length=0.03 radius=0.13
- link BR: geometry visual cylinder length=0.03 radius=0.13
- link FL: geometry visual cylinder length=0.03 radius=0.13
- link FR: geometry visual cylinder length=0.03 radius=0.13
- link base_link: geometry collision box size=0.4 0.4 0.04; visual box size=0.4 0.4 0.04

Commit message: création de la trajectoire

File: controleDrone/urdf/drone.urdf (robot description, URDF)
Before this commit: robot myDrone, 5 links, 4 joints
Links:
- link base_link: geometry collision box size=0.4 0.4 0.04; visual box size=0.2 0.2 0.04
